File: elec/src/bq24045dsqr/elec/layout/default/bq24045dsqr.kicad_pcb (KiCad board)
At the start: 2 copper layers, 225.7 x 100.8 mm, 4 parts

Commit message: fixed maybe
Parts:
- moved C2 34.2 mm to (175.2, 121.3), turned to 90 degrees
- moved C1 32.1 mm to (171.8, 121.3), turned to 90 degrees
- moved U1 31.6 mm to (173.5, 120.6), turned to 180 degrees
- moved R1 30.8 mm to (175.2, 119.4), turned to -90 degrees
Routing:
- net 10: track 0.00 -> 21.4 mm
- net ic-vcc: track 6.47 -> 8.02 mm
- net ic-gnd: track 4.50 -> 5.43 mm
